File: cc2652r_rev_e.brd (EAGLE design)
At the start: 26.4 x 16.8 mm, 41 parts, among them IC3 CC2652R1FRGZ, Y1 Q22FA12800150, Y2 32.768KHz

Commit message: Add files via upload
Parts:
- removed C20, C22: CAP0402, discretes-dev:CAPC1005X40N
- C10, C3, C9: value CAP0402 -> 1pF
- C19, C4: value CAP0402 -> 12pF
- C21: value CAP0402 -> 1.8pF
- L3, L4: value IND0402IND0402 -> 2.4nH
- L5, L6: value IND0402IND0402 -> 2nH
- R2: value RES0402 -> 2.2k
- moved C10 0.56 mm to (19.6, 5.52), turned to 270 degrees
- moved G 0.06 mm to (18.6, 0.90)
Connections:
- net GND: no longer C20.1, C22.2
- net X48M_N: no longer C22.1
- net X48M_P: no longer C20.2
Routing:
- net X48M_N: track 4.26 -> 2.39 mm
- net X48M_P: track 5.50 -> 4.42 mm
- net 13: track 28.9 -> 29.5 mm, vias 1 -> 2
- net 0: track 10.5 -> 9.91 mm
- net 7: track 28.4 -> 28.9 mm, vias 1 -> 2
- net GND: vias 122 -> 136
