File: ipx/cc2652r_rev_e_ipx.brd (EAGLE design)
At the start: 26.4 x 16.8 mm, 39 parts, among them IC3 CC2652R1FRGZ, Y1 Q22FA12800150, Y2 32.768KHz

Commit message: Add files via upload
Parts:
- removed C21: 1.8pF, discretes-dev:CAPC1005X40N
- removed E1: ANTENNA-GROUNDEDTRACE-15.2MM, SparkFun-RF:TRACE_ANTENNA_2.4GHZ_15.2MM
- removed TP1: TPTP06SQ, testpad:TP05SQ
- removed TP2: TPSQTP15SQ, testpad:TP15SQ
- added J4: U.FL, SparkFun-Connectors:U.FL
- moved C19 2.33 mm to (21.4, 8.79)
- moved L6 1.78 mm to (21.0, 7.35), turned to 0 degrees
- moved C10 0.92 mm to (19.1, 6.32), turned to 180 degrees
- moved L5 0.42 mm to (19.1, 7.35)
- moved C1 0.38 mm to (4.17, 14.4)
- moved C12 0.38 mm to (9.33, 15.5)
- moved C13 0.38 mm to (10.2, 4.01)
- moved C17 0.38 mm to (11.2, 4.01)
- moved C18 0.38 mm to (15.0, 5.16)
- moved C2 0.38 mm to (3.14, 14.4)
- moved C3 0.38 mm to (17.3, 8.88)
- moved C4 0.38 mm to (17.3, 4.70)
- moved C8 0.38 mm to (7.80, 14.7)
- moved IC3 0.38 mm to (11.1, 9.86)
- moved J2 0.38 mm to (16.4, 17.2)
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Connections:
- removed net N$9: C21.2, E1.ANT
- net GND: now also J4.1, J4.2; no longer E1.GND
- net N$8: now also J4.FEED; no longer C21.1
Routing:
- net N$9: track 0.96 -> 0.00 mm
- net GND: track 2.04 -> 1.85 mm, vias 136 -> 169
Other:
- board size 26.4 x 16.8 mm -> 23.5 x 16.8 mm

Commit message: Add files via upload
Parts:
- moved J4 9.02 mm to (21.4, 2.87), turned to 90 degrees
- moved C19 2.86 mm to (21.4, 5.93), turned to 270 degrees
- moved R2 1.45 mm to (15.9, 2.73)
- moved G 1.35 mm to (17.7, 2.30), turned to 270 degrees
Routing:
- net 7: track 28.9 -> 27.4 mm, vias 2 -> 1
- net N$7: track 1.08 -> 1.61 mm
- net GND: vias 169 -> 168
Other:
- board text removed: "G"

Commit message: Add files via upload
Parts:
- moved C10 2.83 mm to (20.5, 8.79), turned to 90 degrees
Routing:
- net GND: vias 168 -> 159

Commit message: Add files via upload
Parts:
- added BME280: BME280, bosch-bme280:BME280
- added C25: 100n, ok-discretes-dev:_PKG_C_0402
- added R3, R4: 4.7k, discretes-dev:RESC1005X40N
Connections:
- net 4: now also BME280.4, R3.1
- net 5: now also BME280.3, R4.1
- net GND: now also BME280.1, BME280.5, BME280.7, C25.2
- net VCC: now also BME280.2, BME280.6, BME280.8, C25.1, R3.2, R4.2
Routing:
- net VCC: track 11.8 -> 45.5 mm, vias 3 -> 5
- net 5: track 14.9 -> 26.2 mm, vias 1 -> 2
- net 4: track 14.2 -> 24.1 mm, vias 1 -> 2
- net GND: track 1.85 -> 10.6 mm, vias 159 -> 103
