File: ipx/cc2652r_rev_e_ipx.sch (EAGLE design)
At the start: 36 parts, among them IC3 CC2652R1FRGZ, J4 U.FL, Y1 Q22FA12800150, Y2 32.768KHz

Commit message: Add files via upload
Parts:
- added BME280: BME280, bosch-bme280:BME280
- added C25: 100n, ok-discretes-dev:CAP-0402
- added R3, R4: 4.7k, discretes-dev:RES0402
Connections:
- net 4: now also BME280.SCK, R3.1
- net 5: now also BME280.SDI, R4.1
- net GND: now also BME280.GND, BME280.SDO, C25.2
- net VCC: now also BME280.CSB, BME280.VDD, BME280.VDDIO, C25.1, R3.2, R4.2
